Commit message: Do first adaption for Gazebo Ignition.

File: model/eduard/eduard.urdf (robot description, URDF)
Before this commit: robot $(arg robot_name), 11 links, 10 joints
Links:
- removed link chassis
- removed link imu
- removed link lidar
- removed link motor_a
- removed link motor_b
- removed link motor_c
- removed link motor_d
- removed link range_front_left
- removed link range_front_right
- removed link range_rear_left
- removed link range_rear_right
- added link base_link, mass 5.0; collision box size=0.38 0.22 0.02; collision box size=0.38 0.22 0.02
Joints:
- removed joint axis_front_left
- removed joint axis_front_right
- removed joint axis_rear_left
- removed joint axis_rear_right
- removed joint mount_imu
- removed joint mount_lidar
- removed joint mount_range_front_left
- removed joint mount_range_front_right
- removed joint mount_range_rear_left
- removed joint mount_range_rear_right

Commit message: added red eduard, changed trancparency

File: model/eduard/eduard.urdf (robot description, URDF)
Before this commit: robot $(arg robot_name), 1 links, 0 joints
Links:
- link base_link: geometry collision box size=0.38 0.22 0.02; collision box size=0.38 0.22 0.02
