Commit message: changed paths from uArm package to edu_sim package

File: model/uArm/urdf/model.urdf (robot description, URDF)
Before this commit: robot firefighter, 11 links, 10 joints
Links:
- link add_1: geometry visual mesh filename=package://edu_simulation/model/uArm/urdf/daes/add_1.dae
- link add_2: geometry visual mesh filename=package://edu_simulation/model/uArm/urdf/daes/add_2.dae
- link add_3: geometry visual mesh filename=package://edu_simulation/model/uArm/urdf/daes/add_3.dae
- link add_4: geometry visual mesh filename=package://edu_simulation/model/uArm/urdf/daes/add_4.dae
- link add_5: geometry visual mesh filename=package://edu_simulation/model/uArm/urdf/daes/add_5.dae
- link base: geometry visual mesh filename=package://edu_simulation/model/uArm/urdf/daes/base.STL
- link base_rot: geometry visual mesh filename=package://edu_simulation/model/uArm/urdf/daes/base_rot.dae
- link link_1: geometry visual mesh filename=package://edu_simulation/model/uArm/urdf/daes/link_1.dae
- link link_2: geometry visual mesh filename=package://edu_simulation/model/uArm/urdf/daes/link_2.dae
- link link_3: geometry visual mesh filename=package://edu_simulation/model/uArm/urdf/daes/link_3_2.dae
- link link_end: geometry visual mesh filename=package://edu_simulation/model/uArm/urdf/daes/link_end_2.dae
