Commit message: added uarm part-file and launchfile

File: model/uArm/urdf/uarm_part.xacro (robot description, xacro)
@@ -1,5 +1,4 @@
 <?xml version="1.0"?>
-<robot  xmlns:xacro="http://www.ros.org/wiki/xacro" name="firefighter" >
-<xacro:property name="width" value=".2" />
+<robot xmlns:xacro="http://www.ros.org/wiki/xacro">
   <link name="uarm_base">
     <visual>
