Commit message: fixed args from eduard

File: model/uArm/eduard_uarm.urdf.xacro (robot description, xacro)
@@ -1,13 +1,14 @@
 <?xml version="1.0"?>
 <robot xmlns:xacro="http://www.ros.org/wiki/xacro" name="eduard_uarm">
-  <!-- Eduard (dein bestehendes Modell) -->
+  <!-- Args, die eduard.urdf erwartet -->
+  <xacro:arg name="robot_name" default="eduard"/>
+  <xacro:arg name="wheel_type" default="mecanum"/>
+  <xacro:arg name="eduard_color" default="blue"/>
   <xacro:include filename="$(find edu_simulation)/model/eduard/eduard.urdf"/>
-  <!-- uArm (als Part) -->
-  <xacro:include filename="$(find edu_simulation)/model/uArm/urdf/uarm_part.urdf.xacro"/>
-  <!-- Mount: Eduard base_link -> uArm uarm_base -->
+  <xacro:include filename="$(find edu_simulation)/model/uArm/urdf/uarm_part.xacro"/>
   <joint name="uarm_mount" type="fixed">
     <parent link="base_link"/>
     <child link="uarm_base"/>
-    <origin xyz="0.0 0.0 0.25" rpy="0 0 0"/>
+    <origin xyz="0 0 0.25" rpy="0 0 0"/>
   </joint>
 </robot>
